Commit message: Move gazebo color tags to main urdf files rename gazebo xacro file to be more specific

File: urdf/reggiebot.urdf.xacro (robot description, xacro)
@@ -2,5 +2,5 @@
 <robot xmlns:xacro="http://www.ros.org/wiki/xacro" name="reggiebot">
   <xacro:include filename="reggiebot_core.xacro" />
-  <xacro:include filename="reggiebot_gazebo.xacro" />
+  <xacro:include filename="reggiebot_gazebo_control.xacro" />
   <xacro:include filename="reggiebot_lidar.xacro" />
 </robot>

File: urdf/reggiebot_core.xacro (robot description, xacro)
@@ -60,4 +60,7 @@
     </xacro:inertial_box>
   </link>
+  <gazebo reference="chassis">
+    <material>Gazebo/White</material>
+  </gazebo>
   <!-- LEFT WHEEL LINK -->
   <joint name="left_wheel_joint" type="continuous">
@@ -85,4 +88,7 @@
     </xacro:inertial_cylinder>
   </link>
+  <gazebo reference="left_wheel">
+    <material>Gazebo/Blue</material>
+  </gazebo>
   <!-- RIGHT WHEEL LINK -->
   <joint name="right_wheel_joint" type="continuous">
@@ -110,4 +116,7 @@
     </xacro:inertial_cylinder>
   </link>
+  <gazebo reference="right_wheel">
+    <material>Gazebo/Blue</material>
+  </gazebo>
   <!-- CASTER WHEEL LINK -->
   <joint name="caster_wheel_joint" type="fixed">
@@ -134,3 +143,9 @@
     </xacro:inertial_sphere>
   </link>
+  <gazebo reference="caster_wheel">
+    <material>Gazebo/Grey</material>
+    <!-- make caster wheel "frictionless" (TODO: for now) -->
+    <mu1 value="0.001" />
+    <mu2 value="0.001" />
+  </gazebo>
 </robot>

File: urdf/reggiebot_gazebo_control.xacro (robot description, xacro)
@@ -1,25 +1,4 @@
 <?xml version="1.0"?>
 <robot xmlns:xacro="http://www.ros.org/wiki/xacro">
-  <!-- Colors -->
-  <gazebo reference="chassis">
-    <material>Gazebo/White</material>
-  </gazebo>
-  <gazebo reference="left_wheel">
-    <material>Gazebo/Blue</material>
-  </gazebo>
-  <gazebo reference="right_wheel">
-    <material>Gazebo/Blue</material>
-  </gazebo>
-  <gazebo reference="caster_wheel">
-    <material>Gazebo/Grey</material>
-  </gazebo>
-  <gazebo reference="laser_frame">
-    <material>Gazebo/Black</material>
-  </gazebo>
-  <!-- make caster wheel "frictionless" (TODO: for now) -->
-  <gazebo reference="caster_wheel">
-    <mu1 value="0.001" />
-    <mu2 value="0.001" />
-  </gazebo>
   <!-- basic diff drive plugin, will be replaced with ros2_control -->
   <gazebo>

File: urdf/reggiebot_lidar.xacro (robot description, xacro)
@@ -26,4 +26,7 @@
     </xacro:inertial_cylinder>
   </link>
+  <gazebo reference="laser_frame">
+    <material>Gazebo/Black</material>
+  </gazebo>
   <!-- gazebo ray sensor with ros plugin -->
   <gazebo reference="laser_frame">
